File: DCD/Subcircuits/switches.kicad_sch (KiCad schematic)
At the start: 7 parts

Commit message: Progress on the layout
Parts:
- removed TP3: TestPoint, TestPoint:TestPoint_Pad_D1.5mm, symbol Connector:TestPoint
Connections:
- net GND renamed AGND
Changed lines of the file:
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@@
 		)
 	)
-	(text_box "The transfer function of the whole system from the Ext_Analog input and DAC outputs to the ADC driver positive output, with the assumption that the internal impedances of the DAC output amplifiers and the external function gen are negligibly small, is given by:\n\nV_+ = (V_1 + V_2) * R_f / (R + 2*R_l), where\n\nV_+ is the positive output of the ADC driver\nV_1 is the output of the opamp connected to the output of the DAC\nV_2 is the external input (Ext_Analog)\nR_f is the feedback resistor of the ADC driver\nR are the values of the summing resistors connected in series with the DAC's opamp output and the external input\nR_l is the resistor between the input of the ADC driver and the node summing the currects from the DAC and the external input"
+	(text_box ".\n"
 		(exclude_from_sim no)
 		(at 15.24 77.47 0)
@@
 		)
 	)
-	(text_box "If we set V_- to 0, R_f = R, and R_l = 0, then the voltage measured by the ADC is equal to:\n\nV_o = V_1 + V_2\ncreating a perfect summing amplifier.\n\nThe value of 1kΩ was chosen for the resistor R and capacitors were added in parallel with it to create a low pass filter with cutoff of 1.6MHz. A filter with the same cutoff frequency was reproduced after the DAC driver to create a sharper cutoff."
+	(text_box "."
 		(exclude_from_sim no)
 		(at 15.24 104.14 0)
@@
 	)
 	(junction
-		(at 175.26 46.99)
-		(diameter 0)
-		(color 0 0 0 0)
-	)
-	(junction
 		(at 35.56 63.5)
 		(diameter 0)
@@
 	(wire
 		(pts
-			(xy 175.26 44.45) (xy 175.26 46.99)
-		)
-		(stroke
-			(width 0)
-			(type default)
-		)
-	)
-	(wire
-		(pts
-			(xy 172.72 46.99) (xy 175.26 46.99)
+			(xy 172.72 46.99) (xy 177.8 46.99)
 		)
 		(stroke
@@
 		(pts
 			(xy 123.19 30.48) (xy 123.19 35.56)
-		)
-		(stroke
-			(width 0)
-			(type default)
-		)
-	)
-	(wire
-		(pts
-			(xy 175.26 46.99) (xy 177.8 46.99)
 		)
 		(stroke
@@
 		)
 	)
-	(hierarchical_label "GND"
+	(hierarchical_label "AGND"
 		(shape output)
 		(at 35.56 66.04 270)
@@
 		)
 	)
-	(symbol
-		(lib_id "Connector:TestPoint")
-		(at 175.26 44.45 0)
-		(unit 1)
-		(exclude_from_sim no)
-		(in_bom yes)
-		(on_board yes)
-		(dnp no)
-		(property "Reference" "TP3"
-			(at 173.228 35.56 0)
-			(effects
-				(font
-					(size 1.27 1.27)
-				)
-				(justify left)
-			)
-		)
-		(property "Value" "TestPoint"
-			(at 170.942 38.1 0)
-			(effects
-				(font
-					(size 1.27 1.27)
-				)
-				(justify left)
-			)
-		)
-		(property "Footprint" "TestPoint:TestPoint_Pad_D1.5mm"
-			(at 180.34 44.45 0)
-			(effects
-				(font
-					(size 1.27 1.27)
-				)
-				(hide yes)
-			)
-		)
-		(property "Datasheet" "~"
-			(at 180.34 44.45 0)
-			(effects
-				(font
-					(size 1.27 1.27)
-				)
-				(hide yes)
-			)
-		)
-		(property "Description" "test point"
-			(at 175.26 44.45 0)
-			(effects
-				(font
-					(size 1.27 1.27)
-				)
-				(hide yes)
-			)
-		)
-		(pin "1"
-		)
-		(instances
-			(project "DCD"
-				(path "/b8e3d55b-fa56-4199-88ad-60cfd98f56f9/9d251ce4-04d4-4800-ac42-9fd9e9a8cf74"
-					(reference "TP3")
-					(unit 1)
-				)
-			)
-		)
-	)

Commit message: Progrezz
Other:
- note removed: "Theory of Operation"
Changed lines of the file:
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@@
-		)
-	)
-	(text "Theory of\nOperation"
-		(exclude_from_sim no)
-		(at 168.402 91.44 0)
-		(effects
-			(font
-				(size 3.81 3.81)
-				(thickness 0.762)
-				(bold yes)
-			)
 		)
 	)
