File: DCD/Subcircuits/switches.kicad_sch (KiCad schematic)
At the start: 6 parts

Commit message: Added components part numbers and stuff. Added termination resistors
Parts:
- R17: Order number (none) -> 667-ERA-3AEB470V; Part number  (none) -> ERA-3AEB470V; Supplier (none) -> Mouser
Changed lines of the file:
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@@
+			)
+		)
+		(property "Order number" " 667-ERA-3AEB470V "
+			(at 45.72 57.15 0)
+			(effects
+				(font
+					(size 1.27 1.27)
+				)
+				(hide yes)
+			)
+		)
+		(property "Part number " " ERA-3AEB470V "
+			(at 45.72 57.15 0)
+			(effects
+				(font
+					(size 1.27 1.27)
+				)
+				(hide yes)
+			)
+		)
+		(property "Supplier" "Mouser"
+			(at 45.72 57.15 0)
+			(effects
+				(font
+					(size 1.27 1.27)
+				)
+				(hide yes)
 			)
 		)

Commit message: Added bodges
Parts:
- added C70: 1µF, Capacitor_SMD:C_0603_1608Metric, symbol Device:C
- added FB18: 470Ω, Inductor_SMD:L_0603_1608Metric, symbol Device:FerriteBead_Small
- added R23, R24: 10k, Resistor_SMD:R_0603_1608Metric, symbol Device:R
- added R25: 100, Resistor_SMD:R_0603_1608Metric, symbol Device:R
- R18, R19, R20: value 1k -> 10k; Link (none) -> https://eu.mouser.com/ProductDetail/Panasonic/ERJ-3EKF1002V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; Link  https://www.mouser.com/ProductDetail/Panasonic/ERA-3VRW1001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 -> (none); Order number 667-ERA-3VRW1001V -> 667-ERJ-3EKF1002V; Part number ERA-3VRW1001V -> ERJ-3EKF1002V
Connections:
- net ADC0: now also R18.2, R20.2; no longer R18.1
- net ADC1: now also R23.1, R24.2; no longer R20.1
- net AGND: now also C70.2
- net DAC1: now also R23.2; no longer R20.2
- net at JP2.1 (A): now also R18.1; no longer R18.2
- new net: FB18.2, R25.1
- new net VRR: FB18.1
- new net VRRR: C70.1, R20.1, R24.1, R25.2
Other:
- note removed: "Voltage summing node and a jumper to skip it for using the DAC as an external generator and testing the DAC alone."

Commit message: Bodges
Changed lines of the file:
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@@
 	)
 	(hierarchical_label "VRR"
-		(shape output)
+		(shape input)
 		(at 34.29 113.03 180)
 		(effects
