File: DCD/Subcircuits/adc.kicad_sch (KiCad schematic)
At the start: 42 parts, among them U6 ADR4550BRZ, U7 ADA4945-1ACPZ-R2, U8 ADA4945-1ACPZ-R2, U9 AD4630-24BBCZ

Commit message: Progress on the layout
Parts:
- removed C20, C21, C22, C23, C26: 100p, Capacitor_SMD:C_0603_1608Metric, symbol Device:C_Small
- removed C24: 1µF, Capacitor_SMD:C_0603_1608Metric, symbol Device:C
- removed C25, C34, C35: 1nF, Capacitor_SMD:C_0603_1608Metric, symbol Device:C
- removed R1, R2, R3, R4, R5, R6, R7, R8, R9: 1k, Resistor_SMD:R_0603_1608Metric, symbol Device:R
- removed R12, R13: 100, Resistor_SMD:R_0603_1608Metric, symbol Device:R
- removed U7, U8: ADA4945-1ACPZ-R2, LFCSP16_ADA4945-1ACPZ-R2_ADI, symbol custom_components:ADA4945-1ACPZ-R2
- added FB20: 470Ω, Inductor_SMD:L_0603_1608Metric, symbol Device:FerriteBead_Small
Connections:
- net IN0: now also R14.1
- net IN1: now also R15.1
- net at U9.F1 (IN1+): now also C37.1, R15.2
- net at C36.1, R14.2: now also U9.B1 (IN0+); no longer U9.C1 (IN0-)
- net GND renamed AGND
- net AGND: now also U9.C1 (IN0-), U9.G1 (IN1-), FB20.1; no longer U9.B6 (IOGND), U9.B7 (IOGND), U9.C6 (IOGND), U9.D6 (IOGND), U9.E6 (IOGND), U9.E7 (IOGND), U9.F6 (IOGND), U9.G6 (IOGND), U9.H8 (IOGND)
- new net DGND: FB20.2, U9.B6 (IOGND), U9.B7 (IOGND), U9.C6 (IOGND), U9.D6 (IOGND), U9.E6 (IOGND), U9.E7 (IOGND), U9.F6 (IOGND), U9.G6 (IOGND), U9.H8 (IOGND)
- no-connect marks 14 -> 12
Other:
- moved on the sheet: C27, C28, C29, C30, C31, C32, C33, C36, C37, FB10, FB7, FB8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

Commit message: Schematics for the clock reconditioning
Parts:
- added FB22, FB23, FB24: 470Ω, Inductor_SMD:L_0603_1608Metric, symbol Device:FerriteBead_Small
Connections:
- net 1.8V: now also FB23.2; no longer U9.G3 (VDD_1.8V), U9.H3 (VDD_1.8V)
- net 5V: now also FB24.2; no longer U9.A3 (VDD_5V), U9.B3 (VDD_5V)
- net VIO: now also FB22.2; no longer R16.1, U9.A8 (VIO), U9.B8 (VIO)
- new net: FB24.1, U9.A3 (VDD_5V), U9.B3 (VDD_5V)
- new net: FB22.1, R16.1, U9.A8 (VIO), U9.B8 (VIO)
- new net: FB23.1, U9.G3 (VDD_1.8V), U9.H3 (VDD_1.8V)

Commit message: Added components part numbers and stuff. Added termination resistors
Parts:
- R14: Order number (none) -> 667-ERA-3VEB1000V; Part number (none) -> ERA-3VEB1000V; Supplier (none) -> Mouser
Changed lines of the file:
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@@
+			)
+		)
+		(property "Order number" " 667-ERA-3VEB1000V "
+			(at 58.42 138.43 90)
+			(effects
+				(font
+					(size 1.27 1.27)
+				)
+				(hide yes)
+			)
+		)
+		(property "Part number" " ERA-3VEB1000V"
+			(at 58.42 138.43 90)
+			(effects
+				(font
+					(size 1.27 1.27)
+				)
+				(hide yes)
+			)
+		)
+		(property "Supplier" "Mouser"
+			(at 58.42 138.43 90)
+			(effects
+				(font
+					(size 1.27 1.27)
+				)
+				(hide yes)
 			)
 		)

Commit message: Changed the supplier of the ADC to mouser
Parts:
- U9: Link (none) -> https://eu.mouser.com/ProductDetail/Analog-Devices/AD4630-2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; Order number 505-AD4630-24BBCZ-ND -> 584-AD463024BBCZ; Part number AD4630-24BBCZ -> AD4630-24BBCZ; Supplier DigiKey -> Mouser
Changed lines of the file:
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@@
 			)
 		)
-		(property "Part number" "AD4630-24BBCZ"
+		(property "Part number" " AD4630-24BBCZ"
 			(at 195.58 55.88 0)
 			(effects
@@
 			)
 		)
-		(property "Order number" "505-AD4630-24BBCZ-ND"
+		(property "Order number" " 584-AD463024BBCZ"
 			(at 195.58 55.88 0)
 			(effects
@@
 			)
 		)
-		(property "Supplier" "DigiKey"
+		(property "Supplier" "Mouser"
 			(at 195.58 55.88 0)
 			(effects
+				(font
+					(size 1.27 1.27)
+				)
+				(hide yes)
+			)
+		)
+		(property "Link" "https://eu.mouser.com/ProductDetail/Analog-Devices/AD4630-24BBCZ?qs=Rp5uXu7WBW8YQOXZpUyzpg%3D%3D"
+			(at 195.58 55.88 0)
+			(effects

Commit message: Added bodges
Connections:
- net VRR: now reaches C29.1, FB7.1, FB8.1, U6.6 (VOUT)
Changed lines of the file:
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@@
+	)
+	(junction
+		(at 85.09 35.56)
+		(diameter 0)
+		(color 0 0 0 0)
 	)
 	(junction
@@
 	(wire
 		(pts
+			(xy 85.09 35.56) (xy 100.33 35.56)
+		)
+		(stroke
+			(width 0)
+			(type default)
+		)
+	)
+	(wire
+		(pts
 			(xy 59.69 55.88) (xy 59.69 60.96)
 		)
@@
 	(wire
 		(pts
+			(xy 85.09 25.4) (xy 85.09 35.56)
+		)
+		(stroke
+			(width 0)
+			(type default)
+		)
+	)
+	(wire
+		(pts
 			(xy 259.08 120.65) (xy 259.08 123.19)
 		)
@@
 		(pts
 			(xy 195.58 69.85) (xy 187.96 69.85)
-		)
-		(stroke
-			(width 0)
-			(type default)
-		)
-	)
-	(wire
-		(pts
-			(xy 85.09 35.56) (xy 100.33 35.56)
 		)
 		(stroke
@@
 		(effects
 			(font
+				(size 1.27 1.27)
+			)
+			(justify left)
+		)
+	)
+	(hierarchical_label "VRR"
+		(shape output)
+		(at 85.09 25.4 90)
+		(effects
+			(font
