File: DCD/DCD.kicad_sch (KiCad schematic)
At the start: 9 parts

Commit message: Added bodges
Other:
- sheet ADC ports: added VRR; removed none
- sheet DAC ports: added none; removed DGND
Changed lines of the file:
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@@
-	)
-	(junction
-		(at 144.78 39.37)
-		(diameter 0)
-		(color 0 0 0 0)
 	)
 	(junction
@@
 	(wire
 		(pts
-			(xy 137.16 34.29) (xy 137.16 41.91)
+			(xy 140.97 34.29) (xy 140.97 41.91)
 		)
 		(stroke
@@
 	(wire
 		(pts
-			(xy 82.55 49.53) (xy 82.55 39.37)
-		)
-		(stroke
-			(width 0)
-			(type default)
-		)
-	)
-	(wire
-		(pts
 			(xy 80.01 44.45) (xy 123.19 44.45)
 		)
@@
 	(wire
 		(pts
-			(xy 59.69 72.39) (xy 59.69 80.01)
-		)
-		(stroke
-			(width 0)
-			(type default)
-		)
-	)
-	(wire
-		(pts
-			(xy 144.78 39.37) (xy 144.78 41.91)
+			(xy 58.42 72.39) (xy 58.42 80.01)
 		)
 		(stroke
@@
 	(wire
 		(pts
-			(xy 57.15 72.39) (xy 57.15 80.01)
+			(xy 55.88 72.39) (xy 55.88 80.01)
 		)
 		(stroke
@@
 	(wire
 		(pts
-			(xy 132.08 41.91) (xy 132.08 36.83)
+			(xy 135.89 41.91) (xy 135.89 36.83)
+		)
+		(stroke
+			(width 0)
+			(type default)
+		)
+	)
+	(wire
+		(pts
+			(xy 64.77 72.39) (xy 64.77 80.01)
+		)
+		(stroke
+			(width 0)
+			(type default)
+		)
+	)
+	(wire
+		(pts
+			(xy 138.43 34.29) (xy 138.43 41.91)
+		)
+		(stroke
+			(width 0)
+			(type default)
+		)
+	)
+	(wire
+		(pts
+			(xy 96.52 72.39) (xy 96.52 80.01)
+		)
+		(stroke
+			(width 0)
+			(type default)
+		)
+	)
+	(wire
+		(pts
+			(xy 71.12 72.39) (xy 71.12 80.01)
+		)
+		(stroke
+			(width 0)
+			(type default)
+		)
+	)
+	(wire
+		(pts
+			(xy 59.69 34.29) (xy 59.69 41.91)
+		)
+		(stroke
+			(width 0)
+			(type default)
+		)
+	)
+	(wire
+		(pts
+			(xy 57.15 36.83) (xy 135.89 36.83)
+		)
+		(stroke
+			(width 0)
+			(type default)
+		)
+	)
+	(wire
+		(pts
+			(xy 151.13 34.29) (xy 151.13 80.01)
+		)
+		(stroke
+			(width 0)
+			(type default)
+		)
+	)
+	(wire
+		(pts
+			(xy 144.78 72.39) (xy 144.78 80.01)
+		)
+		(stroke
+			(width 0)
+			(type default)
+		)
+	)
+	(wire
+		(pts
+			(xy 99.06 72.39) (xy 99.06 80.01)
+		)
+		(stroke
+			(width 0)
+			(type default)
+		)
+	)
+	(wire
+		(pts
+			(xy 80.01 46.99) (xy 119.38 46.99)
 		)
 		(stroke
@@
 	(wire
 		(pts
-			(xy 134.62 34.29) (xy 134.62 41.91)
-		)
-		(stroke
-			(width 0)
-			(type default)
-		)
-	)
-	(wire
-		(pts
-			(xy 96.52 72.39) (xy 96.52 80.01)
-		)
-		(stroke
-			(width 0)
-			(type default)
-		)
-	)
-	(wire
-		(pts
-			(xy 74.93 72.39) (xy 74.93 80.01)
-		)
-		(stroke
-			(width 0)
-			(type default)
-		)
-	)
-	(wire
-		(pts
-			(xy 59.69 34.29) (xy 59.69 41.91)
-		)
-		(stroke
-			(width 0)
-			(type default)
-		)
-	)
-	(wire
-		(pts
-			(xy 82.55 39.37) (xy 144.78 39.37)
-		)
-		(stroke
-			(width 0)
-			(type default)
-		)
-	)
-	(wire
-		(pts
-			(xy 57.15 36.83) (xy 132.08 36.83)
-		)
-		(stroke
-			(width 0)
-			(type default)
-		)
-	)
-	(wire
-		(pts
-			(xy 151.13 34.29) (xy 151.13 80.01)
-		)
-		(stroke
-			(width 0)
-			(type default)
-		)
-	)
-	(wire
-		(pts
-			(xy 144.78 72.39) (xy 144.78 80.01)
-		)
-		(stroke
-			(width 0)
-			(type default)
-		)
-	)
-	(wire
-		(pts
-			(xy 99.06 72.39) (xy 99.06 80.01)
-		)
-		(stroke
-			(width 0)
-			(type default)
-		)
-	)
-	(wire
-		(pts
-			(xy 80.01 46.99) (xy 119.38 46.99)
-		)
-		(stroke
-			(width 0)
-			(type default)
-		)
-	)
-	(wire
-		(pts
-			(xy 69.85 72.39) (xy 69.85 80.01)
-		)
-		(stroke
-			(width 0)
-			(type default)
-		)
-	)
-	(wire
-		(pts
 			(xy 85.09 34.29) (xy 85.09 80.01)
 		)
@@
 	(wire
 		(pts
-			(xy 64.77 72.39) (xy 64.77 80.01)
+			(xy 62.23 72.39) (xy 62.23 80.01)
 		)
 		(stroke
@@
 	(wire
 		(pts
-			(xy 144.78 34.29) (xy 144.78 39.37)
+			(xy 82.55 34.29) (xy 82.55 49.53)
 		)
 		(stroke
@@
 		)
 		(pin "3.3V" input
-			(at 134.62 41.91 90)
+			(at 138.43 41.91 90)
 			(effects
 				(font
@@
 		)
 		(pin "7V" input
-			(at 132.08 41.91 90)
+			(at 135.89 41.91 90)
 			(effects
 				(font
@@
 		)
 		(pin "-1.2V" input
-			(at 137.16 41.91 90)
+			(at 140.97 41.91 90)
 			(effects
 				(font
@@
 				)
 				(justify left)
-			)
-		)
-		(pin "DGND" input
-			(at 144.78 41.91 90)
-			(effects
-				(font
-					(size 1.27 1.27)
-				)
-				(justify right)
 			)
 		)
@@
 		)
 		(pin "BSY" input
-			(at 59.69 80.01 90)
+			(at 58.42 80.01 90)
 			(effects
 				(font
@@
 		)
 		(pin "CNV" output
-			(at 57.15 80.01 90)
+			(at 55.88 80.01 90)
 			(effects
 				(font
@@
 		)
 		(pin "~{CS}" output
-			(at 64.77 80.01 90)
+			(at 62.23 80.01 90)
 			(effects
 				(font
@@
 		)
 		(pin "SCK" output
+			(at 64.77 80.01 90)
+			(effects
+				(font
+					(size 1.27 1.27)
+				)
+				(justify right)
+			)
+		)
+		(pin "SDI" output
 			(at 67.31 80.01 90)
 			(effects
@@
 			)
 		)
-		(pin "SDI" output
-			(at 69.85 80.01 90)
-			(effects
-				(font
-					(size 1.27 1.27)
-				)
-				(justify right)
-			)
-		)
 		(pin "SDO0" input
-			(at 74.93 80.01 90)
+			(at 71.12 80.01 90)
 			(effects
 				(font
@@
 		)
 		(pin "3.3V" output
-			(at 134.62 34.29 270)
+			(at 138.43 34.29 270)
 			(effects
 				(font
@@
 		)
 		(pin "GND" input
-			(at 144.78 34.29 270)
+			(at 82.55 34.29 270)
 			(effects
 				(font
@@
 		)
 		(pin "-1.8V" output
-			(at 137.16 34.29 270)
+			(at 140.97 34.29 270)
 			(effects
 				(font
@@
 		)
 		(pin "~{CS}" input
-			(at 64.77 72.39 270)
+			(at 62.23 72.39 270)
 			(effects
 				(font
@@
 		)
 		(pin "SDI" input
-			(at 69.85 72.39 270)
+			(at 67.31 72.39 270)
 			(effects
 				(font
@@
 		)
 		(pin "SDO0" output
-			(at 74.93 72.39 270)
+			(at 71.12 72.39 270)
 			(effects
 				(font
@@
 		)
 		(pin "SCK" input
-			(at 67.31 72.39 270)
+			(at 64.77 72.39 270)
 			(effects
 				(font
@@
 		)
 		(pin "CNV" input
-			(at 57.15 72.39 270)
+			(at 55.88 72.39 270)
 			(effects
 				(font
@@
 		)
 		(pin "BSY" output
-			(at 59.69 72.39 270)
+			(at 58.42 72.39 270)
 			(effects
 				(font
@@
 			(effects
 				(font
+					(size 1.27 1.27)
+				)
+				(justify right)
+			)
+		)
+		(pin "VRR" output
+			(at 80.01 66.04 0)
+			(effects
+				(font

Commit message: Bodges
Other:
- sheet Switches ports: added VRR; removed none
Changed lines of the file:
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@@
+	(wire
+		(pts
+			(xy 80.01 66.04) (xy 87.63 66.04)
+		)
+		(stroke
+			(width 0)
+			(type default)
+		)
+	)
 	(wire
 		(pts
@@
 			(effects
 				(font
+					(size 1.27 1.27)
+				)
+				(justify left)
+			)
+		)
+		(pin "VRR" input
+			(at 87.63 66.04 180)
+			(effects
+				(font
